File: SoundLab16StepSequencer.kicad_pcb (KiCad board)
At the start: 2 copper layers, 372 parts, among them J9 Conn_01x16_Pin, J9 Jack-DC, Q1 MMBT3904-7-F, Q2 2N3904, Q3 2N3906, Q4 2N3904, SW20 SW_Push, SW21 SW_Push, SW22 SW_Push, SW23 SW_Push, U1 40106, U10 TL082, U11 TL084, U12 CD74HC4067M, U13 CD74HC4067SM, U14 4013, U15 40106, U16 40106, U17 40193, U18 TL082, U19 CD4094, U2 4514, U20 TPS560200, U22 LM1117MP-3.3, U3 40106, U4 4013, U5 40106, U6 40193, U7 TL074, U8 4042, U9 40193

Commit message: init placement/layout
Parts:
- removed C75, C76, C81, C85, C86: 4.7uF, Capacitor_SMD:C_0805_2012Metric
- removed C77, C78, C82, C84, C87: 470nF, Capacitor_SMD:C_0805_2012Metric
- removed C79, C80, C83: 47nF, Capacitor_SMD:C_0603_1608Metric
- removed the J9 at (-33.9, 55.9)
- removed L1: L, Inductor_SMD:L_7.3x7.3_H3.5
- removed R129, R130: 10k, Resistor_SMD:R_0603_1608Metric
- removed R131: 105, Resistor_SMD:R_0603_1608Metric
- removed R132: 20k, Resistor_SMD:R_0603_1608Metric
- removed TP1, TP2, TP3, TP4, TP5: TestPoint, TestPoint:TestPoint_Plated_Hole_D2.0mm
- removed U20: TPS560200, Package_TO_SOT_SMD:SOT-23-5
- removed U22: LM1117MP-3.3, Package_TO_SOT_SMD:SOT-223-3_TabPin2
- added J1: External Start, SynthProjConnectors:PJ-301, F.Cu at (-14.2, -67.0)
- added J2: External Clock Input, SynthProjConnectors:PJ-301, F.Cu at (-4.00, -67.0)
- added J3: Trigger Out, SynthProjConnectors:PJ-301, F.Cu at (-14.2, -55.6)
- added J4: Gate Out, SynthProjConnectors:PJ-301, F.Cu at (-4.00, -55.6)
- added J5: External Clock Output, SynthProjConnectors:PJ-301, F.Cu at (-14.2, -44.3)
- added J6: Sequencer CV3, SynthProjConnectors:PJ-301, F.Cu at (-4.00, -44.3)
- added J7: Sequencer CV2, SynthProjConnectors:PJ-301, F.Cu at (-14.2, -33.0)
- added J8: Sequencer CV1, SynthProjConnectors:PJ-301, F.Cu at (-4.00, -33.0)
- added SW1: SRBV141404, SynthProjConnectors:SRBV141404, F.Cu at (-37.6, -34.4)
- added SW10: SW_SPST, SynthProjConnectors:MTS-103-A01-T0, F.Cu at (191.5, 97.0)
- added SW11: SW_SPST, SynthProjConnectors:MTS-103-A01-T0, F.Cu at (211.5, 97.0)
- added SW12: SW_SPST, SynthProjConnectors:MTS-103-A01-T0, F.Cu at (231.5, 97.0)
- added SW13: SW_SPST, SynthProjConnectors:MTS-103-A01-T0, F.Cu at (251.5, 97.0)
- added SW14: SW_SPST, SynthProjConnectors:MTS-103-A01-T0, F.Cu at (271.5, 97.0)
- added SW15: SW_SPST, SynthProjConnectors:MTS-103-A01-T0, F.Cu at (291.5, 97.0)
- added SW16: SW_SPST, SynthProjConnectors:MTS-103-A01-T0, F.Cu at (311.5, 97.0)
- added SW17: SW_SPST, SynthProjConnectors:MTS-103-A01-T0, F.Cu at (331.5, 97.0)
- added SW18: SW_SPST, SynthProjConnectors:MTS-103-A01-T0, F.Cu at (351.5, 97.0)
- added SW19: SW_SPST, SynthProjConnectors:MTS-103-A01-T0, F.Cu at (371.5, 97.0)
- added SW2: SW_Push_DPDT, SynthProjConnectors:MTS-203-A1-T0, F.Cu at (-82.7, -17.3)
- added SW24: SW_Push_DPDT, SynthProjConnectors:MTS-203-A1-T0, F.Cu at (-68.8, -1.02)
- added SW25: SW_SPDT, SynthProjConnectors:MTS-103-A01-T0, F.Cu at (-82.6, -4.22)
- added SW26: SW_SPDT, SynthProjConnectors:MTS-103-A01-T0, F.Cu at (-82.6, 3.70)
- added SW3: SR2612F-0112-21R0B-D8-N, SynthProjConnectors:SR2612F-0112, F.Cu at (162.4, 177.7)
- added SW4: SW_SPST, SynthProjConnectors:MTS-103-A01-T0, F.Cu at (71.5, 97.0)
- added SW5: SW_SPST, SynthProjConnectors:MTS-103-A01-T0, F.Cu at (91.5, 97.0)
- added SW6: SW_SPST, SynthProjConnectors:MTS-103-A01-T0, F.Cu at (111.5, 97.0)
- added SW7: SW_SPST, SynthProjConnectors:MTS-103-A01-T0, F.Cu at (131.5, 97.0)
- added SW8: SW_SPST, SynthProjConnectors:MTS-103-A01-T0, F.Cu at (151.5, 97.0)
- added SW9: SW_SPST, SynthProjConnectors:MTS-103-A01-T0, F.Cu at (171.5, 97.0)
- J9: moved to B.Cu
- RV52: footprint Potentiometer_THT:Potentiometer_Alps_RK09K_Single_Vertical -> Potentiometer_SMD:Potentiometer_Bourns_TC33X_Vertical
- moved RV37 512.8 mm to (369.5, 162.0)
- moved RV10 502.3 mm to (349.5, 118.0)
- moved RV5 495.2 mm to (369.5, 118.0)
- moved RV11 486.5 mm to (349.5, 140.0)
- moved RV6 478.7 mm to (369.5, 140.0)
- moved RV41 476.4 mm to (329.5, 162.0)
- moved RV39 464.9 mm to (349.5, 162.0)
- moved RV7 453.0 mm to (359.5, 186.6)
- moved RV18 446.9 mm to (309.5, 118.0)
- moved RV45 441.1 mm to (289.5, 162.0)
- moved RV19 431.7 mm to (309.5, 140.0)
- moved RV43 428.9 mm to (309.5, 162.0)
- moved RV14 425.2 mm to (329.5, 118.0)
- moved RV15 409.2 mm to (329.5, 140.0)
- moved RV49 407.3 mm to (249.5, 162.0)
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Connections:
- R50 pad 1: Net-(U12-I15) -> Net-(R50-Pad1)
- R50 pad 2: Net-(R50-Pad2) -> Net-(U12-I15)
- R51 pad 1: Net-(U12-I15) -> Net-(R51-Pad1)
- R51 pad 2: Net-(R51-Pad2) -> Net-(U12-I15)
- R53 pad 1: Net-(U12-I1) -> Net-(R53-Pad1)
- R53 pad 2: Net-(R53-Pad2) -> Net-(U12-I1)
- R58 pad 1: Net-(U12-I13) -> Net-(R58-Pad1)
- R58 pad 2: Net-(R58-Pad2) -> Net-(U12-I13)
- R59 pad 1: Net-(U12-I13) -> Net-(R59-Pad1)
- R59 pad 2: Net-(R59-Pad2) -> Net-(U12-I13)
- R61 pad 1: Net-(U12-I3) -> Net-(R61-Pad1)
- R61 pad 2: Net-(R61-Pad2) -> Net-(U12-I3)
- R66 pad 1: Net-(U12-I11) -> Net-(R66-Pad1)
- R66 pad 2: Net-(R66-Pad2) -> Net-(U12-I11)
- R67 pad 1: Net-(U12-I11) -> Net-(R67-Pad1)
- R67 pad 2: Net-(R67-Pad2) -> Net-(U12-I11)
- R69 pad 1: Net-(U12-I5) -> Net-(R69-Pad1)
- R69 pad 2: Net-(R69-Pad2) -> Net-(U12-I5)
- R74 pad 1: Net-(U12-I9) -> Net-(R74-Pad1)
- R74 pad 2: Net-(R74-Pad2) -> Net-(U12-I9)
- R75 pad 1: Net-(U12-I9) -> Net-(R75-Pad1)
- R75 pad 2: Net-(R75-Pad2) -> Net-(U12-I9)
- R77 pad 1: Net-(U12-I7) -> Net-(R77-Pad1)
- R77 pad 2: Net-(R77-Pad2) -> Net-(U12-I7)
- RV14 pad 2: Net-(R58-Pad2) -> Net-(R59-Pad1)
- RV15 pad 2: Net-(R59-Pad2) -> Net-(R58-Pad1)
- RV16 pad 2: Net-(R60-Pad2) -> Net-(R61-Pad1)
- RV17 pad 2: Net-(R61-Pad2) -> Net-(R60-Pad2)
- RV22 pad 2: Net-(R66-Pad2) -> Net-(R67-Pad1)
- RV23 pad 2: Net-(R67-Pad2) -> Net-(R66-Pad1)
- RV24 pad 2: Net-(R68-Pad2) -> Net-(R69-Pad1)
- RV25 pad 2: Net-(R69-Pad2) -> Net-(R68-Pad2)
- RV30 pad 2: Net-(R74-Pad2) -> Net-(R75-Pad1)
- RV31 pad 2: Net-(R75-Pad2) -> Net-(R74-Pad1)
- RV32 pad 2: Net-(R76-Pad2) -> Net-(R77-Pad1)
- RV33 pad 2: Net-(R77-Pad2) -> Net-(R76-Pad2)
- RV5 pad 2: Net-(R50-Pad2) -> Net-(R51-Pad1)
- RV6 pad 2: Net-(R51-Pad2) -> Net-(R50-Pad1)
- RV8 pad 2: Net-(R52-Pad2) -> Net-(R53-Pad1)
- RV9 pad 2: Net-(R53-Pad2) -> Net-(R52-Pad2)
Other:
- board outline added: 314.9 x 110 mm
- board text added: "3U 62HP Eurorack"

Commit message: routing and placing
Parts:
- removed C56: 1uF, Capacitor_SMD:C_0805_2012Metric
- removed D57: 1N914, Diode_SMD:D_SOD-323F
- removed D59: LED, LED_SMD:LED_0805_2012Metric
- removed R100, R109: 1k, Resistor_SMD:R_0603_1608Metric
- removed R101: 3.9k, Resistor_SMD:R_0603_1608Metric
- removed R102: 6.2k, Resistor_SMD:R_0603_1608Metric
- removed R103: 20k, Resistor_SMD:R_0603_1608Metric
- removed R106: 3k, Resistor_SMD:R_0603_1608Metric
- removed RV52: 1M, Potentiometer_SMD:Potentiometer_Bourns_TC33X_Vertical
- D10, D11, D12, D13, D14, D15, D16, D17, D2, D3, D4, D44, D45, D46, D47, D5, D6, D61, D64, D7, D8, D9: footprint LED_SMD:LED_0805_2012Metric -> LED_THT:LED_D5.0mm
- Q2, Q4: value 2N3904 -> MMBT3904-7-F; footprint Package_TO_SOT_THT:TO-92_Inline -> Package_TO_SOT_SMD:SOT-23-3
- Q3: value 2N3906 -> MMBT3906; footprint Package_TO_SOT_THT:TO-92_Inline -> Package_TO_SOT_SMD:SOT-23-3
- moved D33 423.3 mm to (376.5, 92.0)
- moved D3 420.0 mm to (370.2, 85.5), turned to 0 degrees
- moved SW26 418.9 mm to (297.9, 178.8), turned to 90 degrees
- moved J3 408.2 mm to (320.0, 178.8)
- moved D32 406.3 mm to (356.5, 92.2)
- moved U5 402.6 mm to (274.2, 248.5), turned to 0 degrees
- moved U13 401.3 mm to (302.1, 144.8)
- moved C34 394.2 mm to (144.0, 274.1)
- moved C35 394.2 mm to (147.0, 274.1)
- moved C36 394.2 mm to (150.0, 274.1)
- moved C37 394.2 mm to (153.0, 274.1)
- moved D5 394.0 mm to (350.2, 85.5), turned to 0 degrees
- moved J4 390.6 mm to (308.5, 178.8)
- moved D31 389.3 mm to (336.5, 92.2)
- moved C68 383.7 mm to (210.2, 270.5)
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Connections:
- C44 pad 1: Net-(U4B-R) -> Net-(U14B-R)
- C68 pad 1: Net-(U14B-S) -> Net-(U4B-S)
- J5 pad T: /XCLK -> /VariClock2/Clock_Out
- R120 pad 1: Net-(U14B-S) -> Net-(U4B-S)
- R127 pad 2: /XCLK -> /VariClock2/Clock_Out
- R88 pad 2: Net-(U4B-R) -> Net-(U14B-R)
- SW24 pad 6: Net-(U14B-S) -> Net-(U4B-S)
- U1 pad 1: Net-(C46-Pad2) -> Net-(D53-A)
- U1 pad 12: Net-(D55-K) -> /SequencerClocking/UP
- U1 pad 13: Net-(D50-A) -> Net-(U1-Pad13)
- U1 pad 2: Net-(D52-K) -> Net-(U1-Pad2)
- U1 pad 3: Net-(C47-Pad2) -> Net-(U1-Pad2)
- U1 pad 4: Net-(D53-K) -> /SequencerClocking/DN
- U14 pad 10: /VariClock1/RST -> Net-(U14B-R)
- U14 pad 11: /VariClock1/CLK -> GNDREF
- U14 pad 12: Net-(U14B-D) -> Net-(D51-K)
- U14 pad 13: /VariClock2/Q2 -> Net-(D50-K)
- U14 pad 8: Net-(U14B-S) -> Net-(D48-K)
- U14 pad 9: Net-(U14B-D) -> GNDREF
- U15 pad 1: Net-(D53-A) -> Net-(C46-Pad2)
- U15 pad 10: /SequencerClocking/UP -> Net-(D56-K)
- U15 pad 11: Net-(U15-Pad11) -> Net-(D51-A)
- U15 pad 12: Net-(C67-Pad2) -> Net-(D55-K)
- U15 pad 13: /SequencerRandomGenerator/CLK -> Net-(D50-A)
- U15 pad 2: Net-(U15-Pad2) -> Net-(D52-K)
- U15 pad 3: Net-(U15-Pad2) -> Net-(C47-Pad2)
- U15 pad 4: /SequencerClocking/DN -> Net-(D53-K)
- U15 pad 8: Net-(R92-Pad1) -> Net-(U1-Pad13)
- U15 pad 9: /XCLK -> Net-(D52-A)
- U16 pad 8: Net-(R106-Pad2) -> Net-(C67-Pad2)
- U16 pad 9: Net-(R92-Pad1) -> /SequencerRandomGenerator/CLK
- U3 pad 3: Net-(D39-A) -> Net-(D41-A)
- U3 pad 4: Net-(U3-Pad4) -> Net-(C22-Pad2)
- U4 pad 10: Net-(U4B-R) -> /VariClock1/RST
- U4 pad 11: GNDREF -> /VariClock1/CLK
- U4 pad 12: Net-(D51-K) -> Net-(U4B-D)
- U4 pad 13: Net-(D50-K) -> /VariClock2/Q2
- U4 pad 8: Net-(D48-K) -> Net-(U4B-S)
- U4 pad 9: GNDREF -> Net-(U4B-D)
- U5 pad 10: Net-(D56-K) -> (no net)
- U5 pad 11: Net-(D51-A) -> (no net)
- U5 pad 12: Net-(U15-Pad11) -> (no net)
- U5 pad 13: Net-(D52-A) -> (no net)
- U5 pad 3: Net-(D41-A) -> Net-(D39-A)
- U5 pad 4: Net-(C22-Pad2) -> Net-(U5-Pad4)
- U5 pad 5: Net-(U3-Pad4) -> Net-(U5-Pad4)
Other:
- board text added: "Clock Rate"
