File: VariClock3.kicad_sch (KiCad schematic)
At the start: 24 parts, among them U39 CD74HC4067SM

Commit message: created pcb file, placed parts
Parts:
- gave numbers to parts that had none: 23
- renumbered U39 to U13

Commit message: routed 100%
Parts:
- removed C34, C35: 4.7uF, Capacitor_SMD:C_0805_2012Metric, symbol Device:C
- removed C37: 470nF, Capacitor_SMD:C_0805_2012Metric, symbol Device:C
- removed C38, C39: 47nF, Capacitor_SMD:C_0603_1608Metric, symbol Device:C

Commit message: lots of work... created faceplate
Parts:
- RV36, RV37, RV38, RV39, RV40, RV41, RV42, RV43, RV44, RV45, RV46, RV47, RV48, RV49, RV50, RV51: value 100k -> 50k
Changed lines of the file:
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@@
       (effects (font (size 1.27 1.27)) (justify right))
     )
-    (property "Value" "100k" (at 242.443 63.7032 0)
+    (property "Value" "50k" (at 242.443 63.7032 0)
       (effects (font (size 1.27 1.27)) (justify right))
     )
@@
       (effects (font (size 1.27 1.27)) (justify right))
     )
-    (property "Value" "100k" (at 161.798 112.8268 0)
+    (property "Value" "50k" (at 161.798 112.8268 0)
       (effects (font (size 1.27 1.27)) (justify right))
     )
@@
       (effects (font (size 1.27 1.27)) (justify right))
     )
-    (property "Value" "100k" (at 207.518 112.8268 0)
+    (property "Value" "50k" (at 207.518 112.8268 0)
       (effects (font (size 1.27 1.27)) (justify right))
     )
@@
       (effects (font (size 1.27 1.27)) (justify right))
     )
-    (property "Value" "100k" (at 184.658 112.8268 0)
+    (property "Value" "50k" (at 184.658 112.8268 0)
       (effects (font (size 1.27 1.27)) (justify right))
     )
@@
       (effects (font (size 1.27 1.27)) (justify right))
     )
-    (property "Value" "100k" (at 218.948 63.7032 0)
+    (property "Value" "50k" (at 218.948 63.7032 0)
       (effects (font (size 1.27 1.27)) (justify right))
     )
@@
       (effects (font (size 1.27 1.27)) (justify right))
     )
-    (property "Value" "100k" (at 242.443 112.8268 0)
+    (property "Value" "50k" (at 242.443 112.8268 0)
       (effects (font (size 1.27 1.27)) (justify right))
     )
@@
       (effects (font (size 1.27 1.27)) (justify right))
     )
-    (property "Value" "100k" (at 207.518 63.7032 0)
+    (property "Value" "50k" (at 207.518 63.7032 0)
       (effects (font (size 1.27 1.27)) (justify right))
     )
@@
       (effects (font (size 1.27 1.27)) (justify right))
     )
-    (property "Value" "100k" (at 196.088 112.8268 0)
+    (property "Value" "50k" (at 196.088 112.8268 0)
       (effects (font (size 1.27 1.27)) (justify right))
     )
@@
       (effects (font (size 1.27 1.27)) (justify right))
     )
-    (property "Value" "100k" (at 231.013 112.8268 0)
+    (property "Value" "50k" (at 231.013 112.8268 0)
       (effects (font (size 1.27 1.27)) (justify right))
     )
@@
       (effects (font (size 1.27 1.27)) (justify right))
     )
-    (property "Value" "100k" (at 196.088 63.7032 0)
+    (property "Value" "50k" (at 196.088 63.7032 0)
       (effects (font (size 1.27 1.27)) (justify right))
     )
@@
       (effects (font (size 1.27 1.27)) (justify right))
     )
-    (property "Value" "100k" (at 184.658 63.7032 0)
+    (property "Value" "50k" (at 184.658 63.7032 0)
       (effects (font (size 1.27 1.27)) (justify right))
     )
@@
       (effects (font (size 1.27 1.27)) (justify right))
     )
-    (property "Value" "100k" (at 173.863 63.7032 0)
+    (property "Value" "50k" (at 173.863 63.7032 0)
       (effects (font (size 1.27 1.27)) (justify right))
     )
@@
       (effects (font (size 1.27 1.27)) (justify right))
     )
-    (property "Value" "100k" (at 231.013 63.7032 0)
+    (property "Value" "50k" (at 231.013 63.7032 0)
       (effects (font (size 1.27 1.27)) (justify right))
     )
@@
       (effects (font (size 1.27 1.27)) (justify right))
     )
-    (property "Value" "100k" (at 218.948 112.8268 0)
+    (property "Value" "50k" (at 218.948 112.8268 0)
       (effects (font (size 1.27 1.27)) (justify right))
     )
@@
       (effects (font (size 1.27 1.27)) (justify right))
     )
-    (property "Value" "100k" (at 161.798 63.7032 0)
+    (property "Value" "50k" (at 161.798 63.7032 0)
       (effects (font (size 1.27 1.27)) (justify right))
     )
@@
       (effects (font (size 1.27 1.27)) (justify right))
     )
-    (property "Value" "100k" (at 173.863 112.8268 0)
-      (effects (font (size 1.27 1.27)) (justify right))
-    )
+    (property "Value" "50k" (at 173.863 112.8268 0)
+      (effects (font (size 1.27 1.27)) (justify right))
+    )
